Commit message: fix(description): put base_link on the ground under the feet
The upstream root sat at the head, so the model was half below the
RViz / control panel grid. Lift the head 0.15338 m (lowest point at the
zero pose) and drop the matching Gazebo pin offset.

File: description/gazebo/marty_gazebo_physics.xacro (robot description, xacro)
@@ -9,6 +9,6 @@
     <parent link="world"/>
     <child link="base_link"/>
-    <!-- Feet bottoms sit 0.15338 m below base_link at the zero pose; lift so they rest on the ground. -->
-    <origin xyz="0 0 0.15338" rpy="0 0 0"/>
+    <!-- base_link is already at the feet bottoms (see head joint origin). -->
+    <origin xyz="0 0 0" rpy="0 0 0"/>
   </joint>
   <xacro:macro name="gazebo_foot" params="link">

File: description/robot_description/urdf/robot_description.urdf.xacro (robot description, xacro)
@@ -11,6 +11,7 @@
   <link name="base_link"/>
   <!-- Main Structure -->
+  <!-- Lucy: base_link sits on the ground under the feet (lowest point at the zero pose). -->
   <xacro:fixed name="head" parent="base_link" material="blue" mesh="head">
-    <origin xyz="0 0 0" rpy="0 0 0"/>
+    <origin xyz="0 0 0.15338" rpy="0 0 0"/>
   </xacro:fixed>
   <xacro:fixed name="side_panel_left" parent="head" material="yellow" mesh="side_panel">
